File: HW/TEMP_LOGGER/TEMP_LOGGER.kicad_pcb (KiCad board)
At the start: 2 copper layers, 37 parts, among them J1 Conn_01x02, J2 Conn_01x02_Pin, J3 Conn_01x06, J4 Conn_01x03, Q1 DMP6350S, SW1 SW_Omron_B3FS, U1 STM32F030C8Tx, U2 GD25Q16CSJGR, U3 LMV321, U4 LMV321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

Commit message: Board release V0.0
Parts:
- removed J4: Conn_01x03, SparkFun-Connector:1x03
- removed R7: 10K, Resistor_SMD:R_0805_2012Metric
- removed TP2: TestPoint, TestPoint:TestPoint_Pad_D1.0mm
- removed U5: LMV321, Package_TO_SOT_SMD:SOT-353_SC-70-5
- added C10: 20pF, Capacitor_SMD:C_0805_2012Metric, F.Cu at (133.0, 93.5)
- added C11: 4.3pF, Capacitor_SMD:C_0805_2012Metric, F.Cu at (133.0, 84.5)
- added C12: 4.3pF, Capacitor_SMD:C_0805_2012Metric, F.Cu at (133.0, 87.0)
- added C8: 100nF, Capacitor_SMD:C_0805_2012Metric, F.Cu at (138.0, 69.5)
- added C9: 20pF, Capacitor_SMD:C_0805_2012Metric, F.Cu at (133.0, 89.5)
- added D1: GREEN, LED_SMD:LED_0805_2012Metric, F.Cu at (123.5, 89.3)
- added D2: RED, LED_SMD:LED_0805_2012Metric, F.Cu at (123.5, 95.4)
- added J5: Conn_01x02, Connector_PinHeader_2.54mm:PinHeader_1x02_P2.54mm_Vertical, F.Cu at (170.7, 89.4)
- added J6: USB4105-GF-A-060, SparkFun-Connector:USB-C_16, F.Cu at (147.0, 73.3)
- added R10: 100, Resistor_SMD:R_0805_2012Metric, F.Cu at (134.0, 78.0)
- added R11: 100, Resistor_SMD:R_0805_2012Metric, F.Cu at (134.0, 75.5)
- added R8: 510, Resistor_SMD:R_0805_2012Metric, F.Cu at (123.5, 86.3)
- added R9: 330, Resistor_SMD:R_0805_2012Metric, F.Cu at (123.5, 92.4)
- added SW2: SMD_4.6x2.8mm_h1.9mm, SparkFun-Switch:Push_SMD_4.6x2.8mm, F.Cu at (134.0, 70.2)
- added TP12: MCO, TestPoint:TestPoint_Pad_D1.0mm, F.Cu at (154.5, 93.7)
- added Y1: 8.0MHz H130A-8.000-18-2030-EXT-TR, Crystal:Crystal_SMD_5032-2Pin_5.0x3.2mm, F.Cu at (137.7, 91.5)
- added Y2: 32.768 KHz CC7V-T1A, Crystal:Crystal_SMD_MicroCrystal_CC7V-T1A-2Pin_3.2x1.5mm, F.Cu at (137.0, 85.5)
- C1: value C_Small -> 100nF
- C2, C3: footprint SparkFun-Capacitor:C_0805_2012Metric -> Capacitor_SMD:C_0805_2012Metric
- C4, C5, C6, C7: value 1.0uF -> 100nF; footprint SparkFun-Capacitor:C_0805_2012Metric -> Capacitor_SMD:C_0805_2012Metric
- J1: value Conn_01x02 -> 1.27, 2x5, Male, TH; footprint SparkFun-Connector:1x02 -> Connector_PinHeader_1.27mm:PinHeader_2x05_P1.27mm_Vertical
- J2: value Conn_01x02_Pin -> Conn_01x02
- J3: value Conn_01x06 -> Conn_01x03; footprint SparkFun-Connector:1x06 -> Connector_PinSocket_2.54mm:PinSocket_1x03_P2.54mm_Vertical
- SW1: value SW_Omron_B3FS -> SMD_4.6x2.8mm_h1.9mm; footprint Button_Switch_SMD:SW_SPST_Omron_B3FS-100xP -> SparkFun-Switch:Push_SMD_4.6x2.8mm
- U3, U4: value LMV321 -> LM321; footprint Package_TO_SOT_SMD:SOT-353_SC-70-5 -> Package_TO_SOT_SMD:SOT-23-5
- moved J3 93.5 mm to (170.7, 105.2), turned to 180 degrees
- moved J1 84.6 mm to (171.3, 81.8), turned to 180 degrees
- moved R6 83.4 mm to (165.9, 90.7), turned to 90 degrees
- moved TP11 80.3 mm to (165.5, 102.7)
- moved TP10 76.8 mm to (165.5, 100.2)
- moved TP4 75.6 mm to (157.0, 110.5)
- moved TP1 75.3 mm to (147.0, 110.5)
- moved TP3 72.8 mm to (137.5, 110.5)
- moved R1 72.5 mm to (141.5, 114.5), turned to -90 degrees
- moved U3 72.0 mm to (137.5, 114.5)
- moved C7 71.4 mm to (151.4, 96.5), turned to -90 degrees
- moved U4 70.9 mm to (157.0, 114.5), turned to 0 degrees
- moved J2 68.8 mm to (145.7, 114.8), turned to 90 degrees
- moved R4 65.2 mm to (151.0, 103.5), turned to 90 degrees
- moved R2 63.3 mm to (153.0, 114.5), turned to -90 degrees
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Connections:
- J1 pad 1: VCC -> +3V3
- J1 pad 2: GND -> SWDIO
- J3 pad 2: unconnected-(J3-Pin_2-Pad2) -> USART1_TX
- J3 pad 3: unconnected-(J3-Pin_3-Pad3) -> USART1_RX
- R6 pad 2: Net-(J4-Pin_3) -> BOOT0
- U1 pad 10: THERM_REF -> unconnected-(U1-PA0-Pad10)
- U1 pad 11: THERM_OUT -> LED0
- U1 pad 12: THERM_OFST -> LED1
- U1 pad 20: unconnected-(U1-PB2-Pad20) -> THERM_OUT
- U1 pad 21: unconnected-(U1-PB10-Pad21) -> THERM_OFST
- U1 pad 25: LED0 -> unconnected-(U1-PB12-Pad25)
- U1 pad 26: LED0 -> unconnected-(U1-PB13-Pad26)
- U1 pad 29: unconnected-(U1-PA8-Pad29) -> Net-(U1-PA8)
- U1 pad 3: unconnected-(U1-PC14-Pad3) -> OSC32_IN
- U1 pad 34: unconnected-(U1-PA13-Pad34) -> SWDIO
- U1 pad 37: unconnected-(U1-PA14-Pad37) -> SWDCLK
- U1 pad 4: unconnected-(U1-PC15-Pad4) -> OSC32_OUT
- U1 pad 46: unconnected-(U1-PB9-Pad46) -> BTN_1
- U1 pad 5: unconnected-(U1-PF0-Pad5) -> OSC_IN
- U1 pad 6: unconnected-(U1-PF1-Pad6) -> OSC_OUT
- U3 pad 1: Net-(Q1-D) -> Net-(J2-Pin_1)
- U3 pad 3: THERM_REF -> THERM_OUT
- U3 pad 4: THERM_REF -> THERM_OUT
- U4 pad 1: Net-(J2-Pin_1) -> Net-(J2-Pin_2)
- U4 pad 3: THERM_OUT -> THERM_OFST
- U4 pad 4: THERM_OUT -> THERM_OFST
Routing:
- net TEMP_EN: track 0.00 -> 63.5 mm, vias 0 -> 5
- net GND: track 0.00 -> 47.4 mm, vias 0 -> 26
- net NRST: track 0.00 -> 45.1 mm, vias 0 -> 2
- net FLASH_nWP: track 0.00 -> 32.6 mm
- net BTN_1: track 0.00 -> 29.1 mm, vias 0 -> 2
- net BOOT0: track 0.00 -> 29.1 mm, vias 0 -> 2
- net FLASH_MOSI: track 0.00 -> 28.6 mm, vias 0 -> 4
- net FLASH_MISO: track 0.00 -> 28.3 mm, vias 0 -> 2
- net THERM_OFST: track 0.00 -> 28.2 mm
- net FLASH_SCK: track 0.00 -> 27.3 mm, vias 0 -> 2
- net THERM_OUT: track 0.00 -> 27.0 mm, vias 0 -> 2
- net FLASH_nCS: track 0.00 -> 25.6 mm
- net USART1_TX: track 0.00 -> 24.9 mm
- net USART1_RX: track 0.00 -> 24.1 mm
- net SWDCLK: track 0.00 -> 22.3 mm
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- added copper zone on F.Cu, net +3V3
- added copper zone on B.Cu, net GND
Other:
- board outline added: 57 x 54.5 mm
- board text added: "TL_V0.0 Designed by: Uriel Zazueta July 2024"
