File: HW/TEMP_LOGGER/TEMP_LOGGER.kicad_sch (KiCad schematic)
At the start: 37 parts, among them J1 Conn_01x02, J2 Conn_01x02_Pin, J3 Conn_01x06, J4 Conn_01x03, Q1 DMP6350S, SW1 SW_Omron_B3FS, U1 STM32F030C8Tx, U2 GD25Q16CSJGR, U3 LMV321, U4 LMV321, U5 LMV321, U6 MIC5504-3.3YM5

Commit message: Board release V0.0
Parts:
- removed C4, C5, C6, C7: 1.0uF, SparkFun-Capacitor:C_0805_2012Metric, symbol SparkFun-Capacitor:1.0uF_0805_25V_10%
- removed J1: Conn_01x02, SparkFun-Connector:1x02, symbol SparkFun-Connector:Conn_01x02
- removed J3: Conn_01x06, SparkFun-Connector:1x06, symbol SparkFun-Connector:Conn_01x06
- removed J4: Conn_01x03, SparkFun-Connector:1x03, symbol SparkFun-Connector:Conn_01x03
- removed R7: 10K, Resistor_SMD:R_0805_2012Metric, symbol Device:R_US
- removed SW1: SW_Omron_B3FS, Button_Switch_SMD:SW_SPST_Omron_B3FS-100xP, symbol Switch:SW_Omron_B3FS
- removed TP2: TestPoint, TestPoint:TestPoint_Pad_D1.0mm, symbol Connector:TestPoint
- removed U3, U4, U5: LMV321, Package_TO_SOT_SMD:SOT-353_SC-70-5, symbol Amplifier_Operational:LMV321
- added C10, C9: 20pF, Capacitor_SMD:C_0805_2012Metric, symbol SparkFun-Capacitor:1.0uF_0805_25V_10%
- added C11, C12: 4.3pF, Capacitor_SMD:C_0805_2012Metric, symbol SparkFun-Capacitor:1.0uF_0805_25V_10%
- added C4, C5, C6, C7, C8: 100nF, Capacitor_SMD:C_0805_2012Metric, symbol Device:C_Small
- added D1: GREEN, LED_SMD:LED_0805_2012Metric, symbol Device:LED
- added D2: RED, LED_SMD:LED_0805_2012Metric, symbol Device:LED
- added J1: 1.27, 2x5, Male, TH, Connector_PinHeader_1.27mm:PinHeader_2x05_P1.27mm_Vertical, symbol Connector_Generic:Conn_02x05_Odd_Even
- added J3: Conn_01x03, Connector_PinSocket_2.54mm:PinSocket_1x03_P2.54mm_Vertical, symbol Connector_Generic:Conn_01x03
- added J5: Conn_01x02, Connector_PinHeader_2.54mm:PinHeader_1x02_P2.54mm_Vertical, symbol Connector_Generic:Conn_01x02
- added J6: USB4105-GF-A-060, SparkFun-Connector:USB-C_16, symbol SparkFun-Connector:USB_C_Receptacle
- added R10, R11: 100, Resistor_SMD:R_0805_2012Metric, symbol Device:R_US
- added R8: 510, Resistor_SMD:R_0805_2012Metric, symbol Device:R_US
- added R9: 330, Resistor_SMD:R_0805_2012Metric, symbol Device:R_US
- added SW1, SW2: SMD_4.6x2.8mm_h1.9mm, SparkFun-Switch:Push_SMD_4.6x2.8mm, symbol SparkFun-Switch:SPST_Push_SMD_4.6x2.8mm_h1.9mm
- added TP12: MCO, TestPoint:TestPoint_Pad_D1.0mm, symbol Connector:TestPoint
- added U3, U4: LM321, Package_TO_SOT_SMD:SOT-23-5, symbol Amplifier_Operational:LM321
- added Y1: 8.0MHz H130A-8.000-18-2030-EXT-TR, Crystal:Crystal_SMD_5032-2Pin_5.0x3.2mm, symbol SparkFun-Clock:Crystal
- added Y2: 32.768 KHz CC7V-T1A, Crystal:Crystal_SMD_MicroCrystal_CC7V-T1A-2Pin_3.2x1.5mm, symbol SparkFun-Clock:Crystal
- C1: value C_Small -> 100nF
- C2, C3: footprint SparkFun-Capacitor:C_0805_2012Metric -> Capacitor_SMD:C_0805_2012Metric
- J2: value Conn_01x02_Pin -> Conn_01x02
- TP1, TP10, TP11, TP3, TP4, TP5, TP6, TP7, TP8, TP9: now left out of the parts list
Connections:
- net +3V3: now also C4.1, C5.1, C6.1, C7.1, J1.1 (Pin_1), J5.2 (Pin_2), R11.1
- net BOOT0: now also R6.2, J5.1 (Pin_1)
- net GND: now also C10.2, C11.2, C12.2, C4.2, C5.2, C6.2, C7.2, C9.2, J1.3 (Pin_3), J1.5 (Pin_5), J1.9 (Pin_9), J3.1 (Pin_1), J6.GND, J6.S (SHIELD), R10.2, R8.1, R9.1, SW1.1, SW2.1, U3.2 (V-), U4.2 (V-)
- net LED0: now also U1.11 (PA1), D1.2 (A); no longer U1.25 (PB12), U1.26 (PB13)
- net NRST: now also J1.10 (Pin_10), SW1.2
- net TEMP_EN: now also U3.5 (V+), U4.5 (V+)
- net THERM_OFST: now also U1.21 (PB10), U4.3 (-), U4.4; no longer U1.12 (PA2)
- net THERM_OUT: now also U1.20 (PB2), U3.3 (-), U3.4; no longer U1.11 (PA1)
- net USART1_RX: now also J3.3 (Pin_3)
- net USART1_TX: now also J3.2 (Pin_2)
- net VCC: now also J6.VBUS
- net at J2.2 (Pin_2), R2.1: now also U4.1 (+)
- net at J2.1 (Pin_1), R1.2: now also U3.1 (+)
- net at U1.29 (PA8): now also TP12.1
- net OSC32_IN: now reaches U1.3 (PC14)
- net OSC32_IN: now also C11.1, Y2.1
- net SWDIO: now reaches U1.34 (PA13)
- net SWDIO: now also J1.2 (Pin_2)
- net SWDCLK: now reaches U1.37 (PA14)
- net SWDCLK: now also J1.4 (Pin_4)
- net OSC32_OUT: now reaches U1.4 (PC15)
- net OSC32_OUT: now also C12.1, Y2.2
- net BTN_1: now reaches U1.46 (PB9)
- net BTN_1: now also C8.1, R11.2, SW2.2
- net OSC_IN: now reaches U1.5 (PF0)
- net OSC_IN: now also C9.1, Y1.1
- net OSC_OUT: now reaches U1.6 (PF1)
- net OSC_OUT: now also C10.1, Y1.2
- net THERM_REF: no longer names the net of U1.10 (PA0)
- new net: D2.1 (K), R9.2
- new net: J6.A6 (D+), J6.B6 (D+)
- new net: J6.A7 (D-), J6.B7 (D-)
- new net: J6.A8 (NC), J6.B8 (NC)
- new net: J6.NC1 (NC), J6.NC2 (NC), J6.NC3 (NC)
- new net: C8.2, R10.1
- new net: D1.1 (K), R8.2
- new net LED1: D2.2 (A), U1.12 (PA2)
- no-connect marks 30 -> 26
Other:
- note added: "LEDs"
- note added: "Programming Interface"
- moved on the sheet: C2, C3, J2, Q1, R1, R2, R3, R4, R5, R6, TP1, TP10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
